File: mutron_III_plug_in_board/kicad_docs/mutron_III_plug_in_board.sch (KiCad schematic (older format))
At the start: 46 parts, among them J1 Conn_01x04_Male, J2 Conn_01x04_Male, J3 Conn_01x04_Male, J4 Conn_01x08_Male, J5 HP-BP-LP, Q1 BC857, Q2 BCM847, Q3 BC847, U1 TL072, U2 RC4558, U3 vactrol, U4 vactrol, U5 RC4558

Commit message: update mutron-III pcb
Parts:
- removed C1, C2: 47nF, Capacitor_THT:C_Rect_L7.0mm_W3.5mm_P5.00mm, symbol Device:C
- removed C3, C4, C5, C6: 100nF, Capacitor_SMD:C_0805_2012Metric_Pad1.15x1.40mm_HandSolder, symbol Device:C
- removed D1: 1N914, Diode_SMD:D_SOD-123, symbol Diode:1N914
- removed D2: 1N5225B, Diode_SMD:D_SOD-123, symbol Device:D_Zener
- removed Q1: BC857, Package_TO_SOT_SMD:SOT-23_Handsoldering, symbol Transistor_BJT:BC857
- removed Q2: BCM847, mutron_III_plug_in_board:SOT457, symbol my_parts:BCM847DS135
- removed Q3: BC847, Package_TO_SOT_SMD:SOT-23_Handsoldering, symbol Transistor_BJT:BC847
- removed R10, R17: 680k, Resistor_SMD:R_0805_2012Metric_Pad1.15x1.40mm_HandSolder, symbol Device:R
- removed R11, R12, R20, R3: 100k, Resistor_SMD:R_0805_2012Metric_Pad1.15x1.40mm_HandSolder, symbol Device:R
- removed R13, R19: 1k, Resistor_SMD:R_0805_2012Metric_Pad1.15x1.40mm_HandSolder, symbol Device:R
- removed R14, R16, R18: 15k, Resistor_SMD:R_0805_2012Metric_Pad1.15x1.40mm_HandSolder, symbol Device:R
- removed R15: 33k, Resistor_SMD:R_0805_2012Metric_Pad1.15x1.40mm_HandSolder, symbol Device:R
- removed R21: 220k, Resistor_SMD:R_0805_2012Metric_Pad1.15x1.40mm_HandSolder, symbol Device:R
- removed R22: 7k5, Resistor_SMD:R_0805_2012Metric_Pad1.15x1.40mm_HandSolder, symbol Device:R
- removed R4, R5, R6: 10k, Resistor_SMD:R_0805_2012Metric_Pad1.15x1.40mm_HandSolder, symbol Device:R
- removed R7, R8: 22k, Resistor_SMD:R_0805_2012Metric_Pad1.15x1.40mm_HandSolder, symbol Device:R
- removed R9: 100, Resistor_SMD:R_0805_2012Metric_Pad1.15x1.40mm_HandSolder, symbol Device:R
- removed RV1: 10k, Potentiometer_THT:Potentiometer_Bourns_3296W_Vertical, symbol Device:R_POT_TRIM
- removed RV2, RV3: 100k, Potentiometer_THT:Potentiometer_Bourns_3296W_Vertical, symbol Device:R_POT_TRIM
- removed U1: TL072, Package_SO:SOIC-8_3.9x4.9mm_P1.27mm, symbol Amplifier_Operational:TL072
- removed unit 1 of U2
- removed unit 3 of U2
- removed U3, U4: vactrol, mutron_III_plug_in_board:vactrol_dual_footprint, symbol Isolator:VTL5C
- removed U5: RC4558, Package_SO:SOIC-8_3.9x4.9mm_P1.27mm, symbol Amplifier_Operational:RC4558
- J1: renamed from J2; value Conn_01x04_Male -> signal_in
- J2: renamed from J1; value Conn_01x04_Male -> cutoff_CV_in
- J3: value Conn_01x04_Male -> signal_out
- J4: value Conn_01x08_Male -> feedback_CV_in_and_PS
- J5: value HP-BP-LP -> mode_select_jumper; footprint Connector_PinHeader_1.27mm:PinHeader_2x03_P1.27mm_Vertical -> Connector_PinHeader_2.54mm:PinHeader_2x03_P2.54mm_Vertical
- R1: value 68k -> 51k
- R2: value 1M -> 100k
Connections:
- net band_pass is gone; now on an unnamed net: J5.3 (Pin_3), U2.7
- net GND: now also R1.1; no longer U2.5 (+)
- net at U2.6 (-): now also R1.2, R2.2
- net filter_core/signal_v_in: now reaches J1.3 (Pin_3), J1.4 (Pin_4)
- net at R2.1: no longer R1.1
- net CV_scaler/raw_CV_in: now reaches J2.3 (Pin_3), J2.4 (Pin_4)
- net feedback_VCA/feedback_CV_in: now reaches J4.3 (Pin_3), J4.4 (Pin_4)
- net high_pass renamed filter_core/low_pass_out
- net low_pass renamed filter_core/high_pass_out
- new net feedback_VCA/band_pass_FB_in: U2.5 (+)
Other:
- note added: "band pass makeup gain"
- note removed: "0mA to 20mA\nflows through \nthe vactrols"
- note removed: "depth trim"
- note removed: "offset trim"
- note removed: "signal in"
- note removed: "signal out"
- note removed: "zener bends feedback CV\nsignal to approximate a \nreverse log response"
- moved on the sheet: J1, J2, J3, J4
