File: mutron_III_plug_in_board/kicad_docs/mutron_III_plug_in_board.kicad_pcb (KiCad board)
At the start: 2 copper layers, 58.4 x 50.8 mm, 46 parts, among them J1 Conn_01x04_Male, J2 Conn_01x04_Male, J3 Conn_01x04_Male, J4 Conn_01x08_Male, J5 HP-BP-LP, Q1 BC857, Q2 BCM847, Q3 BC847, U1 TL072, U2 RC4558, U3 vactrol, U4 vactrol, U5 RC4558

Commit message: update mutron-III pcb
Parts:
- added C7: 100nF, Capacitor_SMD:C_0805_2012Metric_Pad1.15x1.40mm_HandSolder, F.Cu at (148.0, 61.0)
- added C8: 100nF, Capacitor_SMD:C_0805_2012Metric_Pad1.15x1.40mm_HandSolder, F.Cu at (119.4, 84.5)
- added C9: 100nF, Capacitor_SMD:C_0805_2012Metric_Pad1.15x1.40mm_HandSolder, F.Cu at (115.6, 84.5)
- added R23: 10k, Resistor_SMD:R_0805_2012Metric_Pad1.15x1.40mm_HandSolder, F.Cu at (135.6, 77.5)
- added R24: 100, Resistor_SMD:R_0805_2012Metric_Pad1.15x1.40mm_HandSolder, F.Cu at (143.5, 77.5)
- C3: value 100nF -> 100pF
- D1: value 1N914 -> 1N5225B
- D2: value 1N5225B -> 1N914
- J1: value Conn_01x04_Male -> cutoff_CV_in
- J2: value Conn_01x04_Male -> signal_in
- J3: value Conn_01x04_Male -> signal_out
- J4: value Conn_01x08_Male -> feedback_CV_in_and_PS
- J5: value HP-BP-LP -> mode_select_jumper; footprint Connector_PinHeader_1.27mm:PinHeader_2x03_P1.27mm_Vertical -> Connector_PinHeader_2.54mm:PinHeader_2x03_P2.54mm_Vertical
- Q1: value BC857 -> BCM847; footprint Package_TO_SOT_SMD:SOT-23_Handsoldering -> mutron_III_plug_in_board:SOT457
- Q2: value BCM847 -> MMBT3904; footprint mutron_III_plug_in_board:SOT457 -> Package_TO_SOT_SMD:SOT-23_Handsoldering
- Q3: value BC847 -> MMBT3906
- R1: value 68k -> 51k
- R10: value 680k -> 220k
- R11: value 100k -> 220
- R12: value 100k -> 47k
- R13: value 1k -> 15k
- R15: value 33k -> 47k
- R16: value 15k -> 220
- R17: value 680k -> 33k
- R18: value 15k -> 220k
- R19: value 1k -> 7k5
- R2: value 1M -> 100k
- R21: value 220k -> 1M
- R22: value 7k5 -> 100k
- R3: value 100k -> 10k
- R5, R6: value 10k -> 22k
- R7, R8: value 22k -> 680k
- R9: value 100 -> 220k
- U1: value TL072 -> RC4558
- U3: value vactrol -> TL072; footprint mutron_III_plug_in_board:vactrol_dual_footprint -> Package_SO:SOIC-8_3.9x4.9mm_P1.27mm
- U5: value RC4558 -> vactrol; footprint Package_SO:SOIC-8_3.9x4.9mm_P1.27mm -> mutron_III_plug_in_board:vactrol_dual_footprint
- moved C4 54.9 mm to (108.6, 64.8), turned to 270 degrees
- moved C3 48.3 mm to (110.7, 76.8), turned to 0 degrees
- moved R6 43.7 mm to (116.8, 56.1), turned to 270 degrees
- moved C6 40.4 mm to (148.0, 64.8), turned to 270 degrees
- moved R2 40.3 mm to (144.1, 69.2), turned to 90 degrees
- moved R1 40.3 mm to (141.6, 69.2), turned to 90 degrees
- moved R22 32.6 mm to (110.7, 79.4), turned to 0 degrees
- moved R21 29.6 mm to (110.7, 84.5), turned to 180 degrees
- moved C5 29.0 mm to (108.6, 61.0), turned to 270 degrees
- moved R9 27.8 mm to (123.8, 76.8)
- moved R17 26.7 mm to (140.7, 84.5), turned to 0 degrees
- moved R10 26.2 mm to (123.8, 84.5)
- moved U4 25.2 mm to (121.3, 72.4)
- moved U2 24.8 mm to (142.2, 62.9)
- moved R19 24.6 mm to (153.3, 86.4)
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Connections:
- net Net-(J1-Pad3) renamed /CV_scaler/raw_CV_in
- C1 pad 1: /band_pass -> /feedback_VCA/band_pass_FB_in
- C2 pad 1: /low_pass -> /filter_core/low_pass_out
- C3 pad 1: +12V -> Net-(C3-Pad1)
- C3 pad 2: GND -> Net-(C3-Pad2)
- C4 pad 1: GND -> +12V
- C4 pad 2: -12V -> GND
- C5 pad 1: +12V -> GND
- C5 pad 2: GND -> -12V
- C6 pad 1: GND -> +12V
- C6 pad 2: -12V -> GND
- D1 pad 2: Net-(D1-Pad2) -> GND
- D2 pad 2: GND -> Net-(D2-Pad2)
- J2 pad 3: Net-(J2-Pad3) -> /filter_core/signal_v_in
- J2 pad 4: Net-(J2-Pad3) -> /filter_core/signal_v_in
- J4 pad 3: Net-(J4-Pad3) -> /feedback_VCA/feedback_CV_in
- J4 pad 4: Net-(J4-Pad3) -> /feedback_VCA/feedback_CV_in
- J5 pad 1: /high_pass -> /filter_core/low_pass_out
- J5 pad 3: /band_pass -> Net-(J5-Pad3)
- J5 pad 5: /low_pass -> /filter_core/high_pass_out
- Q1 pad 1: Net-(D1-Pad2) -> Net-(Q1-Pad1)
- Q1 pad 2: Net-(D1-Pad1) -> Net-(Q1-Pad2)
- Q1 pad 3: /I_LED -> Net-(Q1-Pad3)
- Q2 pad 3: Net-(Q2-Pad3) -> GND
- Q3 pad 1: Net-(Q3-Pad1) -> Net-(D2-Pad2)
- Q3 pad 2: Net-(Q3-Pad2) -> Net-(D2-Pad1)
- Q3 pad 3: GND -> /filter_core/LED_I_in
- R1 pad 1: Net-(R1-Pad1) -> GND
- R10 pad 1: Net-(C1-Pad2) -> GND
- R10 pad 2: /high_pass -> Net-(Q1-Pad6)
- R11 pad 1: Net-(R11-Pad1) -> GND
- R11 pad 2: Net-(Q2-Pad3) -> Net-(Q1-Pad2)
- R12 pad 1: GND -> Net-(Q1-Pad6)
- R12 pad 2: Net-(Q2-Pad6) -> +12V
- R13 pad 1: GND -> Net-(Q2-Pad2)
- R13 pad 2: Net-(Q2-Pad2) -> Net-(Q1-Pad1)
- R14 pad 1: Net-(Q2-Pad6) -> -12V
- R14 pad 2: +12V -> Net-(Q2-Pad2)
- R15 pad 1: Net-(Q3-Pad2) -> Net-(Q1-Pad3)
- R15 pad 2: Net-(Q2-Pad1) -> +12V
- R16 pad 1: -12V -> GND
- R16 pad 2: Net-(Q3-Pad2) -> Net-(Q1-Pad5)
- R17 pad 1: Net-(C2-Pad2) -> Net-(Q1-Pad5)
- R17 pad 2: /band_pass -> /feedback_VCA/band_pass_FB_in
- R18 pad 1: Net-(Q2-Pad3) -> Net-(Q2-Pad1)
- R18 pad 2: +12V -> -12V
- R19 pad 1: GND -> /feedback_VCA/feedback_CV_in
- R19 pad 2: Net-(Q2-Pad5) -> Net-(D1-Pad1)
- R2 pad 1: Net-(R1-Pad1) -> Net-(J5-Pad3)
- R2 pad 2: Net-(R2-Pad2) -> Net-(R1-Pad2)
- R20 pad 1: Net-(Q2-Pad5) -> Net-(C3-Pad2)
- R20 pad 2: /band_pass -> Net-(R20-Pad2)
- R21 pad 1: Net-(Q3-Pad1) -> Net-(C3-Pad2)
- R21 pad 2: -12V -> Net-(R21-Pad2)
- R22 pad 1: Net-(J4-Pad3) -> Net-(C3-Pad1)
- R22 pad 2: Net-(D2-Pad1) -> Net-(C3-Pad2)
- R3 pad 2: Net-(R1-Pad1) -> /filter_core/signal_v_in
- R4 pad 1: Net-(R4-Pad1) -> Net-(R3-Pad1)
- R4 pad 2: Net-(J2-Pad3) -> /feedback_VCA/band_pass_FB_out
- R5 pad 1: Net-(R4-Pad1) -> /filter_core/low_pass_out
- R5 pad 2: Net-(R11-Pad1) -> Net-(R5-Pad2)
- R6 pad 1: Net-(D1-Pad2) -> /filter_core/high_pass_out
- R6 pad 2: Net-(R3-Pad1) -> Net-(R5-Pad2)
- R7 pad 1: /low_pass -> Net-(C1-Pad2)
- R7 pad 2: Net-(R7-Pad2) -> /filter_core/high_pass_out
- R8 pad 1: /high_pass -> Net-(C2-Pad2)
- R8 pad 2: Net-(R7-Pad2) -> /feedback_VCA/band_pass_FB_in
- R9 pad 1: GND -> /feedback_VCA/band_pass_FB_out
- R9 pad 2: Net-(D1-Pad1) -> Net-(Q1-Pad3)
- RV1 pad 2: Net-(R1-Pad2) -> Net-(R20-Pad2)
- RV2 pad 2: Net-(R2-Pad2) -> Net-(R21-Pad2)
- RV3 pad 1: Net-(D2-Pad1) -> Net-(D1-Pad1)
- RV3 pad 2: Net-(D2-Pad1) -> Net-(D1-Pad1)
- RV3 pad 3: Net-(Q3-Pad1) -> Net-(Q2-Pad1)
- U1 pad 1: Net-(R3-Pad1) -> /filter_core/high_pass_out
- U1 pad 2: Net-(R1-Pad1) -> Net-(R5-Pad2)
- U1 pad 3: GND -> Net-(R3-Pad1)
- U1 pad 5: Net-(Q2-Pad6) -> GND
- U1 pad 6: Net-(Q2-Pad3) -> Net-(C1-Pad2)
- U1 pad 7: Net-(R11-Pad1) -> /feedback_VCA/band_pass_FB_in
- U2 pad 1: /high_pass -> /filter_core/low_pass_out
- U2 pad 2: Net-(R7-Pad2) -> Net-(C2-Pad2)
- U2 pad 3: Net-(R4-Pad1) -> GND
- U2 pad 5: GND -> /feedback_VCA/band_pass_FB_in
- U2 pad 6: Net-(C1-Pad2) -> Net-(R1-Pad2)
- U2 pad 7: /band_pass -> Net-(J5-Pad3)
- U3 pad 1: -12V -> Net-(C3-Pad1)
- U3 pad 2: Net-(U3-Pad2) -> Net-(C3-Pad2)
- U3 pad 3: /high_pass -> GND
- U3 pad 4: Net-(C1-Pad2) -> -12V
- U4 pad 1: Net-(U3-Pad2) -> -12V
- U4 pad 2: /I_LED -> Net-(U4-Pad2)
- U4 pad 3: /band_pass -> /filter_core/high_pass_out
- U4 pad 4: Net-(C2-Pad2) -> Net-(C1-Pad2)
- U5 pad 1: Net-(U5-Pad1) -> Net-(U4-Pad2)
- U5 pad 2: Net-(U5-Pad1) -> /filter_core/LED_I_in
- U5 pad 3: GND -> /feedback_VCA/band_pass_FB_in
- U5 pad 4: -12V -> Net-(C2-Pad2)
Routing:
- net /band_pass: track 115.9 -> 0.00 mm
- net /feedback_VCA/band_pass_FB_in: track 0.00 -> 70.7 mm, vias 0 -> 2
- net /filter_core/high_pass_out: track 0.00 -> 59.8 mm, vias 0 -> 1
- net /low_pass: track 49.6 -> 0.00 mm
- net /filter_core/low_pass_out: track 0.00 -> 48.2 mm
- net /feedback_VCA/band_pass_FB_out: track 0.00 -> 46.7 mm, vias 0 -> 2
- net /high_pass: track 46.3 -> 0.00 mm
- net -12V: track 203.4 -> 164.1 mm, vias 0 -> 1
- net Net-(R3-Pad1): track 43.8 -> 6.89 mm, vias 2 -> 0
- net Net-(C3-Pad1): track 0.00 -> 34.0 mm
- net Net-(R11-Pad1): track 33.8 -> 0.00 mm, vias 2 -> 0
- net Net-(U3-Pad2): track 31.2 -> 0.00 mm
- net +12V: track 138.5 -> 166.2 mm, vias 4 -> 2
- net Net-(Q1-Pad3): track 0.00 -> 27.0 mm, vias 0 -> 2
- net Net-(J4-Pad3): track 22.7 -> 0.00 mm
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Other:
- board text added: "a"
- board text added: "b"
- board text added: "c"
- board text added: "center"
- board text added: "d"
- board text added: "mutron_III_plug_in_board rev 0 2020-08-01"
- board text removed: "mutron_III_plug_in_board rev 0 2019-07-10"
- board text removed: "offset"

Commit message: generate gerbers
Parts:
- renumbered J2 to J1, J1 to J2

Commit message: change zener
Parts:
- D1: value 1N5225B -> MMSZ5225B
Changed lines of the file:
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@@
       (effects (font (size 1 1) (thickness 0.15)))
     )
-    (fp_text value 1N5225B (at 0 2.1) (layer F.Fab)
+    (fp_text value MMSZ5225B (at 0 2.1) (layer F.Fab)
       (effects (font (size 1 1) (thickness 0.15)))
     )
