File: arp_4072_LPF_plug_in_board/kicad_docs/CV_scaler.sch (KiCad schematic (older format))
At the start: 8 parts, among them U3 TL072

Commit message: fix schemo and pcb problems
Parts:
- R32: value 470k -> 120k
Connections:
- net -12V is gone; now on net GND: RV2.3
Changed lines of the file:
@@
 Sheet 3 5
 Title "ARP 4072 LPF"
-Date "2020-07-26"
-Rev "0"
+Date "2020-08-13"
+Rev "1"
 Comp ""
 Comment1 "creativecommons.org/licenses/by/4.0/"
@@
 P 5750 3000
 F 0 "R32" V 5650 3000 50  0000 C CNN
-F 1 "470k" V 5750 3000 50  0000 C CNN
+F 1 "120k" V 5750 3000 50  0000 C CNN
 F 2 "Resistor_SMD:R_0805_2012Metric_Pad1.15x1.40mm_HandSolder" V 5680 3000 50  0001 C CNN
 F 3 "~" H 5750 3000 50  0001 C CNN
@@
 Text Notes 4450 3150 0    50   ~ 0
 offset trim
-$Comp
-L power:-12V #PWR0117
-U 1 1 5F4ACD3D
-P 5000 3150
-F 0 "#PWR0117" H 5000 3250 50  0001 C CNN
-F 1 "-12V" H 5015 3323 50  0000 C CNN
-F 2 "" H 5000 3150 50  0001 C CNN
-F 3 "" H 5000 3150 50  0001 C CNN
-	1    5000 3150
-	-1   0    0    1
-$EndComp
 $Comp
 L power:+12V #PWR0118
@@
 	0    1    1    0
 $EndComp
+$Comp
+L power:GND #PWR0117
+U 1 1 5FAF5663
+P 5000 3150
+F 0 "#PWR0117" H 5000 2900 50  0001 C CNN
+F 1 "GND" H 5005 2977 50  0000 C CNN
+F 2 "" H 5000 3150 50  0001 C CNN
+F 3 "" H 5000 3150 50  0001 C CNN
+	1    5000 3150
+	1    0    0    -1
+$EndComp
 $EndSCHEMATC
