File: 2164_SVF_plug_in_board/kicad_docs/2164SVF.kicad_pcb (KiCad board)
At the start: 2 copper layers, 58.4 x 50.8 mm, 52 parts, among them J1 signal_input, J2 cutoff_CV_input, J3 signal_output, J4 feedback_CV_and_PS, J5 mode_select_jumper, U1 TL072, U2 SSM2164, U3 TL072, U4 TL072

Commit message: change Fcv offset trim resistor
Parts:
- R18: value 270k -> 68k

Commit message: change 2164 SVF zeners
Parts:
- D1, D2: value 6z2 -> 5z1
