File: late_MS20_VCF_plug_in_board/kicad_docs/late_MS20_VCF_plug_in_board.kicad_pcb (KiCad board)
At the start: 2 copper layers, 58.4 x 50.8 mm, 64 parts, among them J1 signal_in, J2 CV_in, J3 signal_out, J4 feedback_CV_and_PS, J5 hp_lp_jumper, Q1 BCM847DS135, Q2 MMBT3904, Q3 MMBT3904, Q4 MMBT3906, Q5 MMBT3906, Q6 MMBT3906, U1 TL072, U2 LM13700, U3 TL072

Commit message: change late MS20 CV scaling
Parts:
- R24: value 20k -> 10k
- R25: value 270k -> 150k
