File: 2164_phasor_plug_in_board/kicad_docs/2164_phasor_plug_in_board.sch (KiCad schematic (older format))
At the start: 85 parts, among them J1 Conn_01x04_Male, J2 Conn_01x04_Male, J3 Conn_01x04_Male, J4 Conn_01x08_Male, U1 TL074, U2 SSM2164, U3 TL074, U4 SSM2164, U5 TL074, U6 TL072

Commit message: update 2164 phasor board
Parts:
- removed C10, C11, C12, C13, C15, C16, C19, C20: 100nF, Capacitor_SMD:C_0805_2012Metric_Pad1.15x1.40mm_HandSolder, symbol Device:C
- removed C14, C17, C21, C23, C4, C6, C8: 560pF, Capacitor_SMD:C_0805_2012Metric_Pad1.15x1.40mm_HandSolder, symbol Device:C
- removed C18, C2, C24, C5, C7, C9: 220pF, Capacitor_SMD:C_0805_2012Metric_Pad1.15x1.40mm_HandSolder, symbol Device:C
- removed C22: 100pF, Capacitor_SMD:C_0805_2012Metric_Pad1.15x1.40mm_HandSolder, symbol Device:C
- removed C25: 220nF, Capacitor_SMD:C_1206_3216Metric_Pad1.42x1.75mm_HandSolder, symbol Device:C
- removed C3: 470pF, Capacitor_SMD:C_0805_2012Metric_Pad1.15x1.40mm_HandSolder, symbol Device:C
- removed D1: BAT48ZFILM, Diode_SMD:D_SOD-123, symbol Diode:BAT48ZFILM
- removed J1, J2, J3: Conn_01x04_Male, Connector_PinHeader_2.54mm:PinHeader_1x04_P2.54mm_Vertical, symbol Connector:Conn_01x04_Male
- removed J4: Conn_01x08_Male, Connector_PinHeader_2.54mm:PinHeader_1x08_P2.54mm_Vertical, symbol Connector:Conn_01x08_Male
- removed R1, R12, R17, R19, R21, R23, R28, R30, R36, R37, R39, R41, R5, R9: 30k, Resistor_SMD:R_0805_2012Metric_Pad1.15x1.40mm_HandSolder, symbol Device:R
- removed R10, R18, R22, R29, R32, R33, R38: 510, Resistor_SMD:R_0805_2012Metric_Pad1.15x1.40mm_HandSolder, symbol Device:R
- removed R11, R7: 100k, Resistor_SMD:R_0805_2012Metric_Pad1.15x1.40mm_HandSolder, symbol Device:R
- removed R13, R14, R24, R25, R43, R44: 10k, Resistor_SMD:R_0805_2012Metric_Pad1.15x1.40mm_HandSolder, symbol Device:R
- removed R15, R16, R26, R27, R45, R46: 20k, Resistor_SMD:R_0805_2012Metric_Pad1.15x1.40mm_HandSolder, symbol Device:R
- removed R20, R35, R6: 15k, Resistor_SMD:R_0805_2012Metric_Pad1.15x1.40mm_HandSolder, symbol Device:R
- removed R31: 270k, Resistor_SMD:R_0805_2012Metric_Pad1.15x1.40mm_HandSolder, symbol Device:R
- removed R34: 4k7, Resistor_SMD:R_0805_2012Metric_Pad1.15x1.40mm_HandSolder, symbol Device:R
- removed R40: 51k, Resistor_SMD:R_0805_2012Metric_Pad1.15x1.40mm_HandSolder, symbol Device:R
- removed R42: 12k, Resistor_SMD:R_0805_2012Metric_Pad1.15x1.40mm_HandSolder, symbol Device:R
- removed R8: 330k, Resistor_SMD:R_0805_2012Metric_Pad1.15x1.40mm_HandSolder, symbol Device:R
- removed RV1: 10k, Potentiometer_THT:Potentiometer_Bourns_3296W_Vertical, symbol Device:R_POT_TRIM
- removed RV2, RV3: 100k, Potentiometer_THT:Potentiometer_Bourns_3296W_Vertical, symbol Device:R_POT_TRIM
- removed unit 1 of U1
- removed unit 2 of U1
- removed unit 4 of U1
- removed unit 5 of U1
- removed U2, U4: SSM2164, Package_SO:SOIC-16_3.9x9.9mm_P1.27mm, symbol 2164_phasor_plug_in_board-rescue:SSM2164-jordans_parts
- removed U3: TL074, Package_SO:SOIC-14_3.9x8.7mm_P1.27mm, symbol Amplifier_Operational:TL074
- removed unit 4 of U5
- removed unit 2 of U5
- removed unit 3 of U5
- removed unit 5 of U5
- removed U6: TL072, Package_SO:SOIC-8_3.9x4.9mm_P1.27mm, symbol Amplifier_Operational:TL072
- added J1: signal_in, Connector_PinHeader_2.54mm:PinHeader_1x04_P2.54mm_Vertical, symbol Connector_Generic:Conn_01x04
- added J2: CV_in, Connector_PinHeader_2.54mm:PinHeader_1x04_P2.54mm_Vertical, symbol Connector_Generic:Conn_01x04
- added J3: signal_out, Connector_PinHeader_2.54mm:PinHeader_1x04_P2.54mm_Vertical, symbol Connector_Generic:Conn_01x04
- added J4: feedback_CV_and_PS, Connector_PinHeader_2.54mm:PinHeader_1x08_P2.54mm_Vertical, symbol Connector_Generic:Conn_01x08
- added R4: 12k, Resistor_SMD:R_0603_1608Metric, symbol Device:R
- C1: value 560pF -> 470p; footprint Capacitor_SMD:C_0805_2012Metric_Pad1.15x1.40mm_HandSolder -> Capacitor_SMD:C_0603_1608Metric
- R1: renamed from R4; footprint Resistor_SMD:R_0805_2012Metric_Pad1.15x1.40mm_HandSolder -> Resistor_SMD:R_0603_1608Metric
- R2: value 510 -> 30k; footprint Resistor_SMD:R_0805_2012Metric_Pad1.15x1.40mm_HandSolder -> Resistor_SMD:R_0603_1608Metric
- R3: footprint Resistor_SMD:R_0805_2012Metric_Pad1.15x1.40mm_HandSolder -> Resistor_SMD:R_0603_1608Metric
- U1, U5: footprint Package_SO:SOIC-14_3.9x8.7mm_P1.27mm -> Package_SO:TSSOP-14_4.4x5mm_P0.65mm
Connections:
- net +12V: now also J4.7 (Pin_7), J4.8 (Pin_8)
- net -12V: now also J4.5 (Pin_5), J4.6 (Pin_6)
- net GND: now also J1.1 (Pin_1), J1.2 (Pin_2), J2.1 (Pin_1), J2.2 (Pin_2), J3.1 (Pin_1), J3.2 (Pin_2), J4.1 (Pin_1), J4.2 (Pin_2); no longer C1.2, U5.3 (+)
- net at R3.2: now also U5.3 (+), R4.1; no longer R2.1
- net at R1.2: now also R3.1, J1.3 (Pin_3), J1.4 (Pin_4)
- net at U5.1, U5.2 (-): now also J3.3 (Pin_3), J3.4 (Pin_4)
- net all_pass_stages/signal_v_in: now reaches U1.8
- net all_pass_stages/signal_v_in: now also C1.1, R2.1
- net feedback_signal: now reaches R2.2
- net feedback_signal: now also C1.2, R1.1, U1.9 (-); no longer C1.1
- new net CV_scaler/raw_CV_in: J2.3 (Pin_3), J2.4 (Pin_4)
- new net all_pass_stages/signal_v_out: R4.2
- new net feedback_VCA/feedback_CV_in: J4.3 (Pin_3), J4.4 (Pin_4)
Other:
- note removed: "2164 protection"
- note removed: "Attribution: two pole phase shifter idea from\nOsamu Hoshuyama\nuserdisk.webry.biglobe.ne.jp/000/024/65/1/Vcph0505.GIF"
- note removed: "CV summer"
- note removed: "depth trim"
- note removed: "feedback CV in\n0V to +2.048V"
- note removed: "feedback VCA"
- note removed: "frequency CV in\n0V to +2.048V"
- note removed: "frequency CV out\n+2V to 0V"
- note removed: "offset trim"
- note removed: "signal in"
- note removed: "signal out"
- moved on the sheet: R1
